Commit message: tuning pid

File: zeus_arm/urdf/zeus_arm.urdf (robot description, URDF)
Before this commit: robot zeus_arm, 7 links, 6 joints
Joints:
- joint joint_2: limit lower=-2.62 upper=2.62 effort=39 velocity=3.19 -> lower=-2.62 upper=2.62 effort=39000 velocity=3.19
- joint joint_3: limit lower=-2.62 upper=2.62 effort=39 velocity=3.19 -> lower=-2.62 upper=2.62 effort=39000 velocity=3.19
- joint joint_4: limit lower=-2.62 upper=2.62 effort=39 velocity=3.19 -> lower=-2.62 upper=2.62 effort=39000 velocity=3.19
